Commit message: Optimize meshes and organize GLB assets by format
Simplify dense meshes, clean degenerate triangles and improve surface normals.
Convert all 783 source meshes to GLB, remove DAE files and keep 405 optional
STL resources in per-model glb/ and stl/ directories. Update all 67 URDFs to
reference GLB without duplicating the model tree.

Fix Panda hand resource references, finger placement and its disconnected
end-effector frame. Correct the malformed Hans E05 joint offset, documenting
that dimension as an inferred typo fix rather than a verified factory value.

Add mesh conversion, export, audit and validation tools, CI checks, model
catalogs, optimization reports and rendered comparisons. Ensure the detailed
optimization report is included instead of being excluded by .gitignore.

Validation: 23 regression tests; 67 URDFs and 201 loaded poses; 1,188 mesh
geometry checks with no errors or degenerate faces; all 783 GLBs pass the
Khronos validator with zero errors and warnings. Asset hashes and documentation
links match. Preserve 235 documented inertia/limit warnings from the source
models without inventing physical parameters.

File: CameraModel/RealSense/RealSense_D405/RealSense_D405.urdf (robot description, URDF)
Before this commit: robot RealSense_D405, 11 links, 10 joints
Links:
- link camera_link: geometry collision box size=0.023 0.042 0.042; visual mesh filename=meshes/glb/d405.glb

File: CameraModel/RealSense/RealSense_D405/RealSense_D405_and_plug.urdf (robot description, URDF)
Before this commit: robot RealSense_D405_and_plug, 12 links, 11 joints
Links:
- link camera_link: geometry collision box size=0.023 0.042 0.042; visual mesh filename=meshes/glb/d405.glb
- link camera_usb_plug_link: geometry collision mesh filename=meshes/glb/plug_collision.glb; visual mesh filename=meshes/glb/plug.glb

File: CameraModel/RealSense/RealSense_D415/RealSense_D415.urdf (robot description, URDF)
Before this commit: robot RealSense_D415, 11 links, 10 joints
Links:
- link camera_link: geometry collision box size=0.02005 0.099 0.023; visual mesh filename=meshes/glb/d415.glb

File: CameraModel/RealSense/RealSense_D415/RealSense_D415_and_plug.urdf (robot description, URDF)
Before this commit: robot RealSense_D415_and_plug, 12 links, 11 joints
Links:
- link camera_link: geometry collision box size=0.02005 0.099 0.023; visual mesh filename=meshes/glb/d415.glb
- link camera_usb_plug_link: geometry collision mesh filename=meshes/glb/plug_collision.glb; visual mesh filename=meshes/glb/plug.glb

File: CameraModel/RealSense/RealSense_D435/RealSense_D435.urdf (robot description, URDF)
Before this commit: robot RealSense_D435, 11 links, 10 joints
Links:
- link camera_link: geometry collision box size=0.02505 0.090 0.025; visual mesh filename=meshes/glb/d435.glb

File: CameraModel/RealSense/RealSense_D435/RealSense_D435_and_plug.urdf (robot description, URDF)
Before this commit: robot RealSense_D435_and_plug, 12 links, 11 joints
Links:
- link camera_link: geometry collision box size=0.02505 0.090 0.025; visual mesh filename=meshes/glb/d435.glb
- link camera_usb_plug_link: geometry collision mesh filename=meshes/glb/plug_collision.glb; visual mesh filename=meshes/glb/plug.glb

File: CameraModel/RealSense/RealSense_D436/RealSense_D436.urdf (robot description, URDF)
Before this commit: robot RealSense_D436, 15 links, 14 joints
Links:
- link camera_link: geometry collision box size=0.02505 0.090 0.025; visual mesh filename=meshes/glb/d436.glb

File: CameraModel/RealSense/RealSense_D436/RealSense_D436_and_plug.urdf (robot description, URDF)
Before this commit: robot RealSense_D436_and_plug, 16 links, 15 joints
Links:
- link camera_link: geometry collision box size=0.02505 0.090 0.025; visual mesh filename=meshes/glb/d436.glb
- link camera_usb_plug_link: geometry collision mesh filename=meshes/glb/plug_collision.glb; visual mesh filename=meshes/glb/plug.glb

File: CameraModel/RealSense/RealSense_D455/RealSense_D455.urdf (robot description, URDF)
Before this commit: robot RealSense_D455, 16 links, 15 joints
Links:
- link camera_link: geometry collision box size=0.026 0.124 0.029; visual mesh filename=meshes/glb/d455.glb

File: CameraModel/RealSense/RealSense_D585/RealSense_D585.urdf (robot description, URDF)
Before this commit: robot RealSense_D585, 20 links, 19 joints
Links:
- link camera_link: geometry collision box size=0.0931 0.182 0.043; visual mesh filename=meshes/glb/d585.glb

File: RobotModel/ABB/IRB1200_5_90/IRB1200_5_90.urdf (robot description, URDF)
Before this commit: robot ABB_IRB1200_5_90, 8 links, 7 joints
Links:
- link Link1: geometry collision mesh filename=Collision/glb/Link1.glb; visual mesh filename=Visual/glb/Link1.glb
- link Link2: geometry collision mesh filename=Collision/glb/Link2.glb; visual mesh filename=Visual/glb/Link2.glb
- link Link3: geometry collision mesh filename=Collision/glb/Link3.glb; visual mesh filename=Visual/glb/Link3.glb
- link Link4: geometry collision mesh filename=Collision/glb/Link4.glb; visual mesh filename=Visual/glb/Link4.glb
- link Link5: geometry collision mesh filename=Collision/glb/Link5.glb; visual mesh filename=Visual/glb/Link5.glb
- link Link6: geometry collision mesh filename=Collision/glb/Link6.glb; visual mesh filename=Visual/glb/Link6.glb
- link base_link: geometry collision mesh filename=Collision/glb/BaseLink.glb; visual mesh filename=Visual/glb/BaseLink.glb

File: RobotModel/ABB/IRB1200_7_70/IRB1200_7_70.urdf (robot description, URDF)
Before this commit: robot ABB_IRB1200_7_70, 8 links, 7 joints
Links:
- link Link1: geometry collision mesh filename=Collision/glb/Link1.glb; visual mesh filename=Visual/glb/Link1.glb
- link Link2: geometry collision mesh filename=Collision/glb/Link2.glb; visual mesh filename=Visual/glb/Link2.glb
- link Link3: geometry collision mesh filename=Collision/glb/Link3.glb; visual mesh filename=Visual/glb/Link3.glb
- link Link4: geometry collision mesh filename=Collision/glb/Link4.glb; visual mesh filename=Visual/glb/Link4.glb
- link Link5: geometry collision mesh filename=Collision/glb/Link5.glb; visual mesh filename=Visual/glb/Link5.glb
- link Link6: geometry collision mesh filename=Collision/glb/Link6.glb; visual mesh filename=Visual/glb/Link6.glb
- link base_link: geometry collision mesh filename=Collision/glb/BaseLink.glb; visual mesh filename=Visual/glb/BaseLink.glb

File: RobotModel/ABB/IRB1600_10_145/IRB1600_10_145.urdf (robot description, URDF)
Before this commit: robot ABB_IRB1600_10_145, 8 links, 7 joints
Links:
- link Link1: geometry collision mesh filename=Collision/glb/Link1.glb; visual mesh filename=Visual/glb/Link1.glb
- link Link2: geometry collision mesh filename=Collision/glb/Link2.glb; visual mesh filename=Visual/glb/Link2.glb
- link Link3: geometry collision mesh filename=Collision/glb/Link3.glb; visual mesh filename=Visual/glb/Link3.glb
- link Link4: geometry collision mesh filename=Collision/glb/Link4.glb; visual mesh filename=Visual/glb/Link4.glb
- link Link5: geometry collision mesh filename=Collision/glb/Link5.glb; visual mesh filename=Visual/glb/Link5.glb
- link Link6: geometry collision mesh filename=Collision/glb/Link6.glb; visual mesh filename=Visual/glb/Link6.glb
- link base_link: geometry collision mesh filename=Collision/glb/BaseLink.glb; visual mesh filename=Visual/glb/BaseLink.glb

File: RobotModel/ABB/IRB1600_6_120/IRB1600_6_120.urdf (robot description, URDF)
Before this commit: robot ABB_IRB1600_6_120, 8 links, 7 joints
Links:
- link Link1: geometry collision mesh filename=Collision/glb/Link1.glb; visual mesh filename=Visual/glb/Link1.glb
- link Link2: geometry collision mesh filename=Collision/glb/Link2.glb; visual mesh filename=Visual/glb/Link2.glb
- link Link3: geometry collision mesh filename=Collision/glb/Link3.glb; visual mesh filename=Visual/glb/Link3.glb
- link Link4: geometry collision mesh filename=Collision/glb/Link4.glb; visual mesh filename=Visual/glb/Link4.glb
- link Link5: geometry collision mesh filename=Collision/glb/Link5.glb; visual mesh filename=Visual/glb/Link5.glb
- link Link6: geometry collision mesh filename=Collision/glb/Link6.glb; visual mesh filename=Visual/glb/Link6.glb
- link base_link: geometry collision mesh filename=Collision/glb/BaseLink.glb; visual mesh filename=Visual/glb/BaseLink.glb

File: RobotModel/ABB/IRB2600_12_165/IRB2600_12_165.urdf (robot description, URDF)
Before this commit: robot ABB_IRB2600_12_165, 8 links, 7 joints
Links:
- link Link1: geometry collision mesh filename=Collision/glb/Link1.glb; visual mesh filename=Visual/glb/Link1.glb
- link Link2: geometry collision mesh filename=Collision/glb/Link2.glb; visual mesh filename=Visual/glb/Link2.glb
- link Link3: geometry collision mesh filename=Collision/glb/Link3.glb; visual mesh filename=Visual/glb/Link3.glb
- link Link4: geometry collision mesh filename=Collision/glb/Link4.glb; visual mesh filename=Visual/glb/Link4.glb
- link Link5: geometry collision mesh filename=Collision/glb/Link5.glb; visual mesh filename=Visual/glb/Link5.glb
- link Link6: geometry collision mesh filename=Collision/glb/Link6.glb; visual mesh filename=Visual/glb/Link6.glb
- link base_link: geometry collision mesh filename=Collision/glb/BaseLink.glb; visual mesh filename=Visual/glb/BaseLink.glb

File: RobotModel/ABB/IRB2600_12_185/IRB2600_12_185.urdf (robot description, URDF)
Before this commit: robot ABB_IRB2600_12_185, 8 links, 7 joints
Links:
- link Link1: geometry collision mesh filename=Collision/glb/Link1.glb; visual mesh filename=Visual/glb/Link1.glb
- link Link2: geometry collision mesh filename=Collision/glb/Link2.glb; visual mesh filename=Visual/glb/Link2.glb
- link Link3: geometry collision mesh filename=Collision/glb/Link3.glb; visual mesh filename=Visual/glb/Link3.glb
- link Link4: geometry collision mesh filename=Collision/glb/Link4.glb; visual mesh filename=Visual/glb/Link4.glb
- link Link5: geometry collision mesh filename=Collision/glb/Link5.glb; visual mesh filename=Visual/glb/Link5.glb
- link Link6: geometry collision mesh filename=Collision/glb/Link6.glb; visual mesh filename=Visual/glb/Link6.glb
- link base_link: geometry collision mesh filename=Collision/glb/BaseLink.glb; visual mesh filename=Visual/glb/BaseLink.glb

File: RobotModel/ABB/IRB4400L_30_243/IRB4400L_30_243.urdf (robot description, URDF)
Before this commit: robot ABB_IRB4400L_30_243, 8 links, 7 joints
Links:
- link Link1: geometry collision mesh filename=Collision/glb/Link1.glb; visual mesh filename=Visual/glb/Link1.glb
- link Link2: geometry collision mesh filename=Collision/glb/Link2.glb; visual mesh filename=Visual/glb/Link2.glb
- link Link3: geometry collision mesh filename=Collision/glb/Link3.glb; visual mesh filename=Visual/glb/Link3.glb
- link Link4: geometry collision mesh filename=Collision/glb/Link4.glb; visual mesh filename=Visual/glb/Link4.glb
- link Link5: geometry collision mesh filename=Collision/glb/Link5.glb; visual mesh filename=Visual/glb/Link5.glb
- link Link6: geometry collision mesh filename=Collision/glb/Link6.glb; visual mesh filename=Visual/glb/Link6.glb
- link base_link: geometry collision mesh filename=Collision/glb/BaseLink.glb; visual mesh filename=Visual/glb/BaseLink.glb

File: RobotModel/ABB/IRB4600_20_250/IRB4600_20_250.urdf (robot description, URDF)
Before this commit: robot ABB_IRB4600_20_250, 8 links, 7 joints
Links:
- link Link1: geometry collision mesh filename=Collision/glb/Link1.glb; visual mesh filename=Visual/glb/Link1.glb
- link Link2: geometry collision mesh filename=Collision/glb/Link2.glb; visual mesh filename=Visual/glb/Link2.glb
- link Link3: geometry collision mesh filename=Collision/glb/Link3.glb; visual mesh filename=Visual/glb/Link3.glb
- link Link4: geometry collision mesh filename=Collision/glb/Link4.glb; visual mesh filename=Visual/glb/Link4.glb
- link Link5: geometry collision mesh filename=Collision/glb/Link5.glb; visual mesh filename=Visual/glb/Link5.glb
- link Link6: geometry collision mesh filename=Collision/glb/Link6.glb; visual mesh filename=Visual/glb/Link6.glb
- link base_link: geometry collision mesh filename=Collision/glb/BaseLink.glb; visual mesh filename=Visual/glb/BaseLink.glb

File: RobotModel/ABB/IRB4600_40_255/IRB4600_40_255.urdf (robot description, URDF)
Before this commit: robot ABB_IRB4600_40_255, 8 links, 7 joints
Links:
- link Link1: geometry collision mesh filename=Collision/glb/Link1.glb; visual mesh filename=Visual/glb/Link1.glb
- link Link2: geometry collision mesh filename=Collision/glb/Link2.glb; visual mesh filename=Visual/glb/Link2.glb
- link Link3: geometry collision mesh filename=Collision/glb/Link3.glb; visual mesh filename=Visual/glb/Link3.glb
- link Link4: geometry collision mesh filename=Collision/glb/Link4.glb; visual mesh filename=Visual/glb/Link4.glb
- link Link5: geometry collision mesh filename=Collision/glb/Link5.glb; visual mesh filename=Visual/glb/Link5.glb
- link Link6: geometry collision mesh filename=Collision/glb/Link6.glb; visual mesh filename=Visual/glb/Link6.glb
- link base_link: geometry collision mesh filename=Collision/glb/BaseLink.glb; visual mesh filename=Visual/glb/BaseLink.glb

File: RobotModel/AE/AIR10_1210/AIR10_1210.urdf (robot description, URDF)
Before this commit: robot AIR10_1210, 8 links, 7 joints
Links:
- link Link1: geometry collision mesh filename=Collision/glb/Link1.glb; visual mesh filename=Visual/glb/Link1.glb
- link Link2: geometry collision mesh filename=Collision/glb/Link2.glb; visual mesh filename=Visual/glb/Link2.glb
- link Link3: geometry collision mesh filename=Collision/glb/Link3.glb; visual mesh filename=Visual/glb/Link3.glb
- link Link4: geometry collision mesh filename=Collision/glb/Link4.glb; visual mesh filename=Visual/glb/Link4.glb
- link Link5: geometry collision mesh filename=Collision/glb/Link5.glb; visual mesh filename=Visual/glb/Link5.glb
- link Link6: geometry collision mesh filename=Collision/glb/Link6.glb; visual mesh filename=Visual/glb/Link6.glb
- link base_link: geometry collision mesh filename=Collision/glb/BaseLink.glb; visual mesh filename=Visual/glb/BaseLink.glb
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